Commit message: modify: urdf corrected

File: kinematics/desky.urdf (robot description, URDF)
Before this commit: robot desky, 7 links, 6 joints
Links:
- removed link link1
- removed link link2
- removed link link3
- removed link link4
- removed link link5
- added link dynamixel1; visual box size=0.047 0.03 0.04
- added link dynamixel2; visual box size=0.047 0.03 0.04
- added link dynamixel3; visual box size=0.047 0.03 0.04
- added link dynamixel4; visual box size=0.047 0.03 0.04
- added link dynamixel5; visual box size=0.047 0.03 0.04
- link base_link: geometry visual box size=0.12 0.12 0.05
Joints:
- joint joint1: child link1 -> dynamixel1; origin xyz=0 0 0.05 rpy=0 0 0 -> xyz=0 0 0.095 rpy=0 0 0
- joint joint2: axis 1 0 0 -> 0 0 1; child link2 -> dynamixel2; origin xyz=0 0 0.03 rpy=0 0 0 -> xyz=-0.01 0 0.02 rpy=0 1.5708 3.1416; parent link1 -> dynamixel1
- joint joint3: axis 0 1 0 -> 0 0 1; child link3 -> dynamixel3; origin xyz=0 0 0.04 rpy=0 0 0 -> xyz=-0.0275 0.02 0.02 rpy=-1.5708 3.1416 0; parent link2 -> dynamixel2
- joint joint4: axis 0 1 0 -> 0 0 1; child link4 -> dynamixel4; origin xyz=0.12 0 0 rpy=0 0 0 -> xyz=0.115 0 0 rpy=0 0 0; parent link3 -> dynamixel3
- joint joint5: axis 0 1 0 -> 0 0 1; child link5 -> dynamixel5; origin xyz=0.10 0 0 rpy=0 0 0 -> xyz=0.115 0 0 rpy=0 0 0; parent link4 -> dynamixel4
- joint tool_joint: parent link5 -> dynamixel5

Commit message: reafactor: refactored app.py

File: kinematics/desky.urdf (robot description, URDF)
Before this commit: robot desky, 7 links, 6 joints
Joints:
- joint joint1: limit lower=-1.5708 upper=1.5708 effort=1.5 velocity=6.0 -> lower=-2.61799 upper=2.61799 effort=1.5 velocity=6.0
- joint joint2: limit lower=-1.5708 upper=1.5708 effort=1.5 velocity=6.0 -> lower=-2.61799 upper=2.61799 effort=1.5 velocity=6.0
- joint joint3: limit lower=-1.5708 upper=1.5708 effort=1.5 velocity=6.0 -> lower=-2.61799 upper=2.61799 effort=1.5 velocity=6.0
- joint joint4: limit lower=-1.5708 upper=1.5708 effort=1.5 velocity=6.0 -> lower=-2.61799 upper=2.61799 effort=1.5 velocity=6.0
- joint joint5: limit lower=-1.5708 upper=1.5708 effort=1.5 velocity=6.0 -> lower=-2.61799 upper=2.61799 effort=1.5 velocity=6.0

Commit message: feat: added mediapipe hands

File: kinematics/desky.urdf (robot description, URDF)
Before this commit: robot desky, 7 links, 6 joints
Joints:
- joint joint2: origin xyz=-0.01 0 0.02 rpy=0 1.5708 3.1416 -> xyz=-0.01 0 0.026 rpy=0 1.5708 3.1416
- joint joint3: origin xyz=-0.0275 0.02 0.02 rpy=-1.5708 3.1416 0 -> xyz=-0.0275 0.02 0.015 rpy=-1.5708 3.1416 0
- joint tool_joint: origin xyz=0.08 0 0 rpy=0 0 0 -> xyz=0.057 0 0 rpy=0 0 0
