Commit message: modify: corrected kinematics

File: kinematics/configure/desky.urdf (robot description, URDF)
Before this commit: robot desky, 14 links, 13 joints
Joints:
- joint base_shell_joint: origin xyz=0 0 0 rpy=0 0 0 -> xyz=0 0 0 rpy=0 0 -1.5708
- joint joint2: limit lower=-1.53589 upper=1.53589 effort=1.5 velocity=6.0 -> lower=-0.13090 upper=0.13090 effort=1.5 velocity=6.0
- joint joint5: limit lower=-3.10669 upper=2.05949 effort=1.5 velocity=6.0 -> lower=-1.57080 upper=1.57080 effort=1.5 velocity=6.0
- joint tool_tip_joint: origin xyz=0 -0.03275 0.401065 rpy=0 0 0 -> xyz=0 -0.03275 0.434 rpy=0 0 0
